File: hw/humidor/humidor.kicad_sch (KiCad schematic)
At the start: 29 parts, among them J1 PWR IN, J2 PWR IN/EXTSENS/IND, J3 IN_SENSOR, J4 Conn_01x05, J5 HEAT/FAN/HS, J6 Conn_01x05_Pin, Q1 2N7002, Q2 IRFD9120, Q3 IRL540, SW1 SW_Push, U1 LT1086-ADJ

Commit message: finalized board with all DRC satisfied. Next step is to try double side layout.
Parts:
- removed J4: Conn_01x05, Connector_PinSocket_2.54mm:PinSocket_1x05_P2.54mm_Vertical, symbol Connector_Generic:Conn_01x05
- added H1, H2, H3, H4: MountingHole, MountingHole:MountingHole_3.5mm, symbol Mechanical:MountingHole
- added JP2: SolderJumper_3_Bridged12, Jumper:SolderJumper-3_P1.3mm_Bridged2Bar12_RoundedPad1.0x1.5mm, symbol Jumper:SolderJumper_3_Bridged12
Connections:
- net +12V: now also JP2.3 (B); no longer J1.1 (Pin_1), J5.1 (Pin_1)
- new net: J1.1 (Pin_1), JP2.1 (A)
- new net HEAT_PWR: J5.1 (Pin_1), JP2.2 (C)
- no-connect marks 34 -> 33
Other:
- moved on the sheet: J2, Q1, Q2, Q3, R6, R7, R8
